File: Hardware/rplink/mcu.kicad_sch (KiCad schematic)
At the start: 1 part, among them U1 Pico

Commit message: rev 0.1
Parts:
- added C14, C15, C16, C20: 104/X7R, Capacitor_SMD:C_0402_1005Metric, symbol Generic:C0402
- added C21, C22: 4.7uF/X7R, Capacitor_SMD:C_0805_2012Metric, symbol Generic:C0805
- added J3, J4: Conn_01x04, Connector_PinHeader_2.54mm:PinHeader_1x04_P2.54mm_Vertical, symbol Connector_Generic:Conn_01x04
- added R20, R28, R29: 100R, Resistor_SMD:R_0402_1005Metric, symbol Generic:R0402
- added R21, R22, R23, R24, R26: 4.7K, Resistor_SMD:R_0402_1005Metric, symbol Generic:R0402
- added R25, R27: 10K, Resistor_SMD:R_0402_1005Metric, symbol Generic:R0402
- added R30: 100K, Resistor_SMD:R_0402_1005Metric, symbol Generic:R0402
- added SW1: SW_SP3T, Button_Switch_SMD:SW_SP3T_PCM13, symbol Switch:SW_SP3T
- added SW2: SW_Push, Button_Switch_SMD:SW_Push_1P1T_NO_CK_KMR2, symbol Switch:SW_Push
- added U8: MX25R3235FM2xx0, Package_SO:SOP-8_5.28x5.23mm_P1.27mm, symbol Memory_Flash:MX25R3235FM2xx0
- added U9: AT24CS64-SSHM, Package_SO:SOIC-8_3.9x4.9mm_P1.27mm, symbol Memory_EEPROM:AT24CS64-SSHM
Connections:
- net M_TXD: now reaches U1.1 (UART0_TX/I2C0_SDA/SPI0_RX/GP0)
- net T_TDI: now reaches U1.10 (I2C1_SCL/SPI0_TX/GP7)
- net T_SWDIO_DIR: now reaches U1.11 (UART1_TX/I2C0_SDA/SPI1_RX/GP8)
- net EE_WP: now reaches U1.12 (UART1_RX/I2C0_SCL/SPI1_CS/GP9)
- net EE_WP: now also R23.1, U9.7 (WP)
- net GND: now reaches U1.13 (GND)
- net GND: now also U1.18 (GND), U1.23 (GND), U1.28 (GND), U1.3 (GND), U1.33 (AGND), U1.38 (GND), U1.42 (GND), U1.8 (GND), C14.2, C15.2, C16.2, C20.2, C21.2, C22.2, J3.3 (Pin_3), J4.1 (Pin_1), R30.1, SW1.3, SW2.2, U8.4 (GND), U9.1 (A0), U9.2 (A1), U9.3 (A2), U9.4 (GND)
- net DF_SCK: now reaches U1.14 (I2C1_SDA/SPI1_SCK/GP10)
- net DF_SCK: now also U8.6 (SCLK)
- net DF_MOSI: now reaches U1.15 (I2C1_SCL/SPI1_TX/GP11)
- net DF_MOSI: now also U8.5 (SI/SIO0)
- net DF_MISO: now reaches U1.16 (UART0_TX/I2C0_SDA/SPI1_RX/GP12)
- net DF_MISO: now also U8.2 (SO/SIO1)
- net ~{DF_CS}: now reaches U1.17 (UART0_RX/I2C0_SCL/SPI1_CS/GP13)
- net ~{DF_CS}: now also R24.2, U8.1 (~{CS})
- net EE_SDA: now reaches U1.19 (I2C1_SDA/SPI1_SCK/GP14)
- net EE_SDA: now also R21.1, U9.5 (SDA)
- net M_RXD: now reaches U1.2 (UART0_RX/I2C0_SCL/SPI0_CSN/GP1)
- net EE_SCL: now reaches U1.20 (I2C1_SCL/SPI1_TX/GP15)
- net EE_SCL: now also R22.1, U9.6 (SCL)
- net TX485: now reaches U1.21 (UART0_TX/I2C0_SDA/SPI0_RX/GP16)
- net TX485: now also J3.2 (Pin_2)
- net RX485: now reaches U1.22 (UART0_RX/I2C0_SCL/SPI0_CS/GP17)
- net RX485: now also J3.1 (Pin_1)
- net at U1.24 (I2C1_SDA/SPI0_SCK/GP18): now also J4.4 (Pin_4)
- net at U1.25 (I2C1_SCL/SPI0_TX/GP19): now also J4.3 (Pin_3)
- net CTRL_5V: now reaches U1.26 (I2C0_SDA/GP20)
- net CTRL_3V3: now reaches U1.27 (I2CO_SCL/GP21)
- net at U1.30 (RUN): now also R29.1
- net at U1.31 (I2C1_SDA/ADC0/GP26): now also C20.1, R20.1
- net at U1.32 (I2C1_SCL/ADC1/GP27): now also C16.1, R28.1
- net +3V3: now reaches U1.36 (3V3)
- net +3V3: now also C14.1, C15.1, C21.1, J4.2 (Pin_2), R21.2, R22.2, R23.2, R24.1, R25.2, U8.3 (~{WP}/SIO2), U8.7 (~{RESET}/SIO3), U8.8 (VCC), U9.8 (VCC)
- net T_TCK_SWCLK: now reaches U1.4 (I2C1_SDA/SPI0_SCK/GP2)
- net +5V: now reaches U1.40 (VBUS)
- net +5V: now also C22.1, J3.4 (Pin_4)
- net T_TMS_SWDIO: now reaches U1.5 (I2C1_SCL/SPI0_TX/GP3)
- net M_SWDIN: now reaches U1.6 (UART1_TX/I2C0_SDA/SPI0_RX/GP4)
- net T_TDO_SWO: now reaches U1.7 (UART1_RX/I2C0_SCL/SPI0_CS/GP5)
- net ~{T_RESET}: now reaches U1.9 (I2C1_SDA/SPI0_SCK/GP6)
- new net: R29.2, SW2.1
- new net: R25.1, R26.1, R28.2, SW1.1
- new net: R26.2, R27.1, SW1.2
- new net: R27.2, R30.2, SW1.4
- new net VTGT_ADIN: R20.2
- no-connect marks 0 -> 7
Other:
- note added: "Not Use"
- note added: "S1 0V TARET S2 1.055V 3.3V S3 1.964V 5V NC 3.036V"
- moved on the sheet: U1
