File: Hardware/rplink/jtag.kicad_sch (KiCad schematic)
At the start: 5 parts, among them U2 74LVC2T45DC

Commit message: rev 0.1
Parts:
- removed C1, C2: C, symbol Device:C
- removed R1, R2: 100R, symbol Device:R
- removed U2: 74LVC2T45DC, Package_SO:VSSOP-8_2.3x2mm_P0.5mm, symbol Logic_LevelTranslator:74LVC2T45DC
- added C1, C10, C11, C12, C15, C16, C2, C20, C21, C22, C3, C4, C46, C5, C6, C7, C8, C9: 104/X7R, Capacitor_SMD:C_0402_1005Metric, symbol Generic:C0402
- added J1: Conn_02x05_Odd_Even, Connector_PinHeader_2.54mm:PinHeader_2x05_P2.54mm_Horizontal, symbol Connector_Generic:Conn_02x05_Odd_Even
- added R1, R10, R11, R12, R13, R14, R17, R18, R2, R20, R21, R22, R3, R30, R4, R5, R57, R58, R59, R6, R7, R8, R9: 100R, Resistor_SMD:R_0402_1005Metric, symbol Generic:R0402
- added R37, R38: 100K NC, Resistor_SMD:R_0402_1005Metric, symbol Generic:R0402
- added U15, U2, U3, U4, U5, U6, U7, U8, U9: SN74LVC1T45DBV, Package_TO_SOT_SMD:SOT-363_SC-70-6_Handsoldering, symbol Logic_LevelTranslator:SN74LVC1T45DBV
Connections:
- net +3V3: now also C1.1, C11.1, C15.1, C20.1, C22.1, C3.1, C6.1, C7.1, C9.1, U15.1 (VCCA), U2.1 (VCCA), U3.1 (VCCA), U4.1 (VCCA), U5.1 (VCCA), U6.1 (VCCA), U7.1 (VCCA), U8.1 (VCCA), U9.1 (VCCA)
- net GND: now also C1.2, C10.2, C11.2, C12.2, C15.2, C16.2, C2.2, C20.2, C21.2, C22.2, C3.2, C4.2, C46.2, C5.2, C6.2, C7.2, C8.2, C9.2, J1.3 (Pin_3), J1.9 (Pin_9), R38.1, U15.2 (GND), U2.2 (GND), U3.2 (GND), U4.2 (GND), U4.5 (DIR), U5.2 (GND), U6.2 (GND), U6.5 (DIR), U7.2 (GND), U8.2 (GND), U8.5 (DIR), U9.2 (GND), U9.5 (DIR)
- net VTGT: now also C10.1, C12.1, C16.1, C2.1, C21.1, C4.1, C46.1, C5.1, C8.1, R37.2, U15.6 (VCCB), U2.6 (VCCB), U3.6 (VCCB), U4.6 (VCCB), U5.6 (VCCB), U6.6 (VCCB), U7.6 (VCCB), U8.6 (VCCB), U9.6 (VCCB)
- new net: R8.2, U4.3 (A)
- new net: R6.1, U4.4 (B)
- new net: R9.2, U5.3 (A)
- new net: R7.1, U5.4 (B)
- new net: R22.2, U5.5 (DIR)
- new net: R13.2, U7.3 (A)
- new net: R30.2, U9.3 (A)
- new net: R18.1, U9.4 (B)
- new net: R57.2, U15.3 (A)
- new net: R59.1, U15.4 (B)
- new net: R58.2, U15.5 (DIR)
- new net: R12.2, U6.3 (A)
- new net: R10.1, U6.4 (B)
- new net: R2.2, U3.3 (A)
- new net: R1.1, R37.1, U3.4 (B)
- new net: R11.1, U7.4 (B)
- new net: R38.2, R4.1, U2.4 (B)
- new net: R21.2, U7.5 (DIR)
- new net: R14.2, U8.3 (A)
- new net: R17.1, U8.4 (B)
- new net: R3.2, U3.5 (DIR)
- new net: R20.2, U2.5 (DIR)
- new net: R5.2, U2.3 (A)
- new net H_RXD: J1.7 (Pin_7), R10.2
- new net H_TCK_SWCLK: J1.4 (Pin_4)
- new net H_TDI: J1.8 (Pin_8)
- new net H_TDO_SWD: J1.6 (Pin_6), R6.2
- new net H_TMS_SWDIO: J1.2 (Pin_2)
- new net H_TXD: J1.5 (Pin_5)
- new net T_RESET_CHK: R30.1
- new net T_RESET_EN: R58.1
- new net T_RXD: R12.1
- new net T_SWDIN: R14.1
- new net T_SWD_OE: R3.1
- new net T_TCK_EN: R20.1
- new net T_TCK_SWCLK: R5.1
- new net T_TCK_SWCLK_H: R4.2
- new net T_TDI: R9.1
- new net T_TDI_EN: R22.1
- new net T_TDI_H: R7.2
- new net T_TDO_SWO: R8.1
- new net T_TMS_SWDIO: R2.1
- new net T_TMS_SWDIO_H: R1.2, R17.2
- new net T_TXD: R13.1
- new net T_TXD_EN: J1.1 (Pin_1), R21.1
- new net T_TXD_H: R11.2
- new net ~{H_RESET}: J1.10 (Pin_10)
- new net ~{T_RESET_H}: R18.2, R59.2
- new net ~{T_RESET}: R57.1
Other:
- note added: "--> DIR = VCC"
- note added: "--> DIR = VCC <-- DIR = GND"
- note added: "<-- DIR = GND"
- note added: "GND"
- note added: "GND/TXD"
- note added: "KEY/RXD"
- note added: "NC/TDI"
- note added: "SWCLK/TCLK"
- note added: "SWDIO/TMS"
- note added: "SWO/TDO"
- note added: "VCC"
- note added: "~{RESET}"

Commit message: 完成初步布局
Parts:
- removed C10, C5, C6, C9: 104/X7R, Capacitor_SMD:C_0402_1005Metric, symbol Generic:C0402
- removed R1, R11, R4, R59, R7: 100R, Resistor_SMD:R_0402_1005Metric, symbol Generic:R0402
- removed R37: 100K NC, Resistor_SMD:R_0402_1005Metric, symbol Generic:R0402
- removed U4, U6, U8, U9: SN74LVC1T45DBV, Package_TO_SOT_SMD:SOT-363_SC-70-6_Handsoldering, symbol Logic_LevelTranslator:SN74LVC1T45DBV
- added R13, R15, R19, R3, R5: 47R, Resistor_SMD:R_0805_2012Metric, symbol Generic:R0805
- added R52, R54, R55, R56, R57, R58: 100K, Resistor_SMD:R_0402_1005Metric, symbol Generic:R0402
- added U4, U8: SN74LVC2T45DCUR, Package_SO:VSSOP-8_2.3x2mm_P0.5mm, symbol Logic_LevelTranslator:SN74LVC2T45DCUR
- R23: renamed from R38; value 100K NC -> 100K
- renumbered C12 to C10, C22 to C11, C46 to C12, C3 to C13, C4 to C14, C20 to C15, C21 to C16, C7 to C3, C8 to C4, C15 to C7, C16 to C8, C11 to C9, R14 to R10, R17 to R11, R13 to R12, R57 to R14, R21 to R16, R58 to R17, R5 to R18, R30 to R20, R18 to R21, R20 to R22, R8 to R24, R6 to R25, R9 to R4, R12 to R6, R10 to R7, R3 to R8, R22 to R9, U3 to U1, U5 to U2, U7 to U5, U15 to U6, U2 to U7
Connections:
- net +3V3: now also U4.1 (VCCA), U8.1 (VCCA)
- net GND: now also R52.1, R54.1, R55.1, R56.1, R57.1, R58.1, U4.4 (GND), U4.5 (DIR), U8.4 (GND), U8.5 (DIR)
- net H_RXD: now also R56.2
- net H_TDO_SWD: now also R58.2
- net T_TCK_SWCLK_H: now also R23.2, R19.2
- net T_TDI_H: now also R5.2, R54.2
- net T_TMS_SWDIO_H: now also R3.2, R52.2
- net T_TXD_EN: no longer J1.1 (Pin_1)
- net T_TXD_H: now also R13.2, R57.2
- net VTGT: now also U4.8 (VCCB), U8.8 (VCCB)
- net ~{T_RESET_H}: now also R15.2, R55.2
- net at R24.2: now also U4.3 (A2)
- net at R25.1: now also U4.6 (B2)
- net at U2.4 (B): now also R5.1
- net at R20.2: now also U8.2 (A1)
- net at R21.1: now also U8.7 (B1)
- net at U6.4 (B): now also R15.1
- net at R6.2: now also U8.3 (A2)
- net at R7.1: now also U8.6 (B2)
- net at U1.4 (B): now also R3.1
- net at U5.4 (B): now also R13.1
- net at U7.4 (B): now also R19.1; no longer R23.2
- net at R10.2: now also U4.2 (A1)
- net at R11.1: now also U4.7 (B1)
- new net VOUT: J1.1 (Pin_1)
Other:
- moved on the sheet: C10, C13, C14, C9, J1, R12, R16, R18, R22, R23, R24, R25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
