File: Hardware/rplink/ps.kicad_sch (KiCad schematic)
At the start: 43 parts, among them J2 USB_C_Receptacle_USB2.0_16P, Q2 CJL2623, Q3 CJL2623, Q4 Q_PMOS_GDS, SW4 SW_SP3T, U1 TPD2S017, U10 LMV321, U11 TPS78233DDC, U17 TPS78233DDC

Commit message: 完成初步布局
Parts:
- removed Q4: Q_PMOS_GDS, Package_TO_SOT_SMD:SOT-23, symbol Device:Q_PMOS_GDS
- added Q1: DMG2301L, Package_TO_SOT_SMD:SOT-23, symbol Transistor_FET:DMG2301L
- Q2, Q3: footprint (none) -> Package_TO_SOT_SMD:SOT-23-6
- U12: renamed from U10; footprint (none) -> Package_TO_SOT_SMD:SOT-23-5
- renumbered C27 to C30, C32 to C31, C29 to C32, C30 to C33, C19 to C34, C28 to C35, C47 to C36, C48 to C39, C31 to C40, C49 to C42, C17 to C45, C50 to C46, C18 to C47, C52 to C48, C13 to C52, C23 to C53, R45 to R26, R46 to R27, R23 to R30, R19 to R31, R31 to R32, R28 to R34, R29 to R35, R24 to R37, R25 to R38, R26 to R42, R27 to R43, R15 to R48, R39 to R49, R16 to R50, R43 to R51, SW4 to SW1, U17 to U10, U1 to U11, U11 to U15
Connections:
- net VBUS: now also Q1.2 (S)
- net VTGT: now also Q1.3 (D)
- net at R31.1, U12.4: now also Q1.1 (G)
Other:
- note added: "Si2301CDS"
