File: Hardware/rplink/rp2404n.kicad_sch (KiCad schematic)
At the start: 38 parts, among them J4 Conn_01x03, J6 Conn_01x04, SW1 SW_Push, SW2 SW_Push, U14 W25Q128JVS, U19 AT24CS64-SSHM, U20 RP2040, Y2 12MHz

Commit message: 完成初步布局
Parts:
- J3: renamed from J6; footprint (none) -> Connector_PinHeader_2.54mm:PinHeader_1x04_P2.54mm_Vertical
- J4: footprint (none) -> Connector_PinHeader_2.54mm:PinHeader_1x03_P2.54mm_Vertical
- SW3: renamed from SW2; footprint Button_Switch_SMD:SW_Push_1P1T_NO_CK_PTS125Sx43PSMTR -> Button_Switch_SMD:SW_Push_1P1T_NO_CK_KMR2
- Y1: renamed from Y2; footprint (none) -> Crystal:Crystal_SMD_WE_CFPX-180-4Pin_3.2x2.5mm
- renumbered C55 to C19, C58 to C20, C59 to C21, C60 to C22, C61 to C23, C62 to C24, C63 to C25, C64 to C26, C66 to C27, C67 to C28, C69 to C29, C68 to C37, C56 to C38, C57 to C41, C54 to C43, C65 to C44, C51 to C49, C53 to C50, C14 to C51, R41 to R28, R42 to R29, R51 to R33, R35 to R36, R53 to R39, R54 to R40, R55 to R41, R36 to R44, R52 to R45, R33 to R46, R34 to R47, SW1 to SW2, U20 to U13, U19 to U14, U14 to U16
Connections:
- net KEY: now also C51.1, R47.2
