File: Hardware/rplink/rplink.kicad_pcb (KiCad board)
At the start: 2 copper layers, 82 x 30 mm, 177 parts, among them J1 Conn_02x05_Odd_Even, J2 USB_C_Receptacle_USB2.0_14P, Q1 MMBT3904, SW1 SW_Push, SW1 SW_SP3T, SW2 SW_Push, SW3 SW_Push, SW4 SW_SP3T, U1 TPD2S017, U11 TPS78233DDC, U14 W25Q128JVS, U15 SN74LVC1T45DBV, U17 TPS78233DDC, U19 AT24CS64-SSHM, U2 SN74LVC1T45DBV, U20 RP2040, U3 SN74LVC1T45DBV, U4 SN74LVC1T45DBV, U5 SN74LVC1T45DBV, U6 SN74LVC1T45DBV, U7 SN74LVC1T45DBV, U8 SN74LVC1T45DBV, U9 SN74LVC1T45DBV

Commit message: 完成初步布局
Parts:
- removed the C10 at (255.3, 70.5)
- removed the C14 at (231.7, 77.9)
- removed the C15 at (204.2, 36.8)
- removed the C16 at (262.4, 50.9)
- removed C17, C18: 4.7uF/X7R, Capacitor_SMD:C_0805_2012Metric
- removed the C19 at (255.1, 48.5)
- removed the C20 at (215.9, 38.5)
- removed the C22 at (192.3, 47.1)
- removed the C26 at (184.2, 37.8)
- removed the C34 at (180.0, 37.5)
- removed the C36 at (180.0, 40.1)
- removed C5, C59, C6: 104/X7R, Capacitor_SMD:C_0402_1005Metric
- removed the C9 at (248.8, 70.6)
- removed the R15 at (273.7, 55.2)
- removed the R16 at (273.7, 56.2)
- removed the R17 at (258.9, 72.4)
- removed the R18 at (260.9, 72.4)
- removed the R20 at (215.9, 37.5)
- removed the R21 at (207.6, 42.2)
- removed the R23 at (208.1, 39.0)
- removed the R25 at (263.4, 54.9)
- removed the R26 at (263.4, 52.9)
- removed the R27 at (263.4, 50.9)
- removed the R28 at (262.4, 52.9)
- removed the R29 at (250.5, 38.5)
- removed the R30 at (263.4, 49.0)
- removed the R31 at (249.4, 45.9)
- removed the R32 at (130.8, 63.4)
- removed the R32 at (245.4, 45.9)
- removed the R33 at (255.1, 46.0)
- removed the R34 at (259.1, 46.0)
- removed the R35 at (257.1, 46.0)
- removed the R36 at (247.4, 45.9)
- removed the R37 at (259.6, 58.9)
- removed the R4 at (259.6, 60.9)
- removed the R40 at (130.8, 67.4)
- removed the R8 at (248.5, 61.7)
- removed the SW2 at (254.6, 39.4)
- removed the SW2 at (130.9, 28.0)
- removed SW4: SW_SP3T, Button_Switch_SMD:SW_SP3T_PCM13
- removed the U10 at (248.7, 48.5)
- removed the U11 at (258.4, 48.4)
- removed the U4 at (252.1, 60.7)
- removed the U6 at (252.0, 70.7)
- added J3: Conn_01x04, Connector_PinHeader_2.54mm:PinHeader_1x04_P2.54mm_Vertical, F.Cu at (222.9, 46.0)
- added J4: Conn_01x03, Connector_PinHeader_2.54mm:PinHeader_1x03_P2.54mm_Vertical, F.Cu at (214.4, 46.1)
- added Q2: CJL2623, Package_TO_SOT_SMD:SOT-23-6, F.Cu at (251.5, 36.8)
- added Q3: CJL2623, Package_TO_SOT_SMD:SOT-23-6, F.Cu at (251.5, 41.2)
- added R52: 100K, Resistor_SMD:R_0402_1005Metric, F.Cu at (249.8, 52.4)
- added R54: 100K, Resistor_SMD:R_0402_1005Metric, F.Cu at (249.2, 64.8)
- added R55: 100K, Resistor_SMD:R_0402_1005Metric, F.Cu at (249.1, 72.5)
- added R56: 100K, Resistor_SMD:R_0402_1005Metric, F.Cu at (248.0, 71.0)
- added R57: 100K, Resistor_SMD:R_0402_1005Metric, F.Cu at (249.4, 60.1)
- added R58: 100K, Resistor_SMD:R_0402_1005Metric, F.Cu at (248.0, 48.3)
- added U12: LMV321, Package_TO_SOT_SMD:SOT-23-5, F.Cu at (271.6, 37.0)
- added Y1: 12MHz, Crystal:Crystal_SMD_WE_CFPX-180-4Pin_3.2x2.5mm, F.Cu at (226.3, 58.5)
- C21: value 4.7uF/X7R -> 104/X7R; footprint Capacitor_SMD:C_0805_2012Metric -> Capacitor_SMD:C_0402_1005Metric
- J2: value USB_C_Receptacle_USB2.0_14P -> USB_C_Receptacle_USB2.0_16P
- Q1: value MMBT3904 -> DMG2301L
- R13: renamed from R11; value 100R -> 47R; footprint Resistor_SMD:R_0402_1005Metric -> Resistor_SMD:R_0805_2012Metric
- R15: renamed from R59; value 100R -> 47R; footprint Resistor_SMD:R_0402_1005Metric -> Resistor_SMD:R_0805_2012Metric
- R19: value 100K -> 47R; footprint Resistor_SMD:R_0402_1005Metric -> Resistor_SMD:R_0805_2012Metric
- R23: renamed from R38; value 100K NC -> 100K
- R24: value 4.7K -> 100R
- R3: renamed from R1; value 100R -> 47R; footprint Resistor_SMD:R_0402_1005Metric -> Resistor_SMD:R_0805_2012Metric
- R5: renamed from R7; value 100R -> 47R; footprint Resistor_SMD:R_0402_1005Metric -> Resistor_SMD:R_0805_2012Metric
- U4: renamed from U8; value SN74LVC1T45DBV -> SN74LVC2T45DCUR; footprint Package_TO_SOT_SMD:SOT-363_SC-70-6_Handsoldering -> Package_SO:VSSOP-8_2.3x2mm_P0.5mm
- U8: renamed from U9; value SN74LVC1T45DBV -> SN74LVC2T45DCUR; footprint Package_TO_SOT_SMD:SOT-363_SC-70-6_Handsoldering -> Package_SO:VSSOP-8_2.3x2mm_P0.5mm
- moved J1 179.6 mm to (264.0, 60.0), turned to 0 degrees
- moved SW3 177.5 mm to (234.7, 71.2)
- moved U13 152.8 mm to (217.5, 57.0), turned to 90 degrees
- moved C35 150.6 mm to (271.6, 32.2)
- moved R31 143.5 mm to (269.3, 36.9), turned to 90 degrees
- moved R32 142.8 mm to (272.1, 40.8), turned to 180 degrees
- moved R30 142.5 mm to (268.5, 39.9), turned to 180 degrees
- moved C34 140.6 mm to (263.5, 37.8), turned to -90 degrees
- moved R28 138.2 mm to (205.3, 55.2)
- moved R29 138.2 mm to (205.3, 56.1)
- moved C36 136.8 mm to (271.2, 33.7)
- moved C42 135.9 mm to (259.5, 56.2), turned to 180 degrees
- moved C40 135.3 mm to (272.1, 39.9), turned to 180 degrees
- moved C39 130.7 mm to (270.3, 39.9)
- moved R49 129.3 mm to (258.2, 43.4), turned to 180 degrees
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- renumbered C12 to C10, C22 to C11, C46 to C12, C3 to C13, C4 to C14, C20 to C15, C21 to C16, C55 to C19, C58 to C20, C60 to C22, C61 to C23, C62 to C24, C63 to C25, C64 to C26, C66 to C27, C67 to C28, C69 to C29, C7 to C3, C27 to C30, C32 to C31, C29 to C32, C30 to C33, C19 to C34, C28 to C35, C47 to C36, C68 to C37, C56 to C38, C48 to C39, C8 to C4, C31 to C40, C57 to C41, C49 to C42, C54 to C43, C65 to C44, C17 to C45, C50 to C46, C18 to C47, C52 to C48, C51 to C49, C53 to C50, C14 to C51, C13 to C52, C23 to C53, C15 to C7, C16 to C8, C11 to C9, R14 to R10, R17 to R11, R13 to R12, R57 to R14, R21 to R16, R58 to R17, R5 to R18, R30 to R20, R18 to R21, R20 to R22, R6 to R25, R45 to R26, R46 to R27, R41 to R28, R42 to R29, R23 to R30, R19 to R31, R31 to R32, R51 to R33, R28 to R34, R29 to R35, R35 to R36, R24 to R37, R25 to R38, R53 to R39, R9 to R4, R54 to R40, R55 to R41, R26 to R42, R27 to R43, R36 to R44, R52 to R45, R33 to R46, R34 to R47, R15 to R48, R39 to R49, R16 to R50, R43 to R51, R12 to R6, R10 to R7, R3 to R8, R22 to R9, SW1 to SW2, U3 to U1, U17 to U10, U1 to U11, U20 to U13, U19 to U14, U11 to U15, U14 to U16, U5 to U2, U7 to U5, U15 to U6, U2 to U7
Connections:
- C21 pad 1: +3V3 -> +1V1
- C51 pad 1: Net-(C14-Pad1) -> /RP2040N/KEY
- J1 pad 1: /JTAG/VOUT -> VOUT
- J2 pad A8: (no net) -> unconnected-(J2-SBU1-PadA8)
- J2 pad B8: (no net) -> unconnected-(J2-SBU2-PadB8)
- Q1 pad 1: Net-(Q1-B) -> Net-(Q1-G)
- Q1 pad 2: GND -> VBUS
- Q1 pad 3: /JTAG/~{T_RESET_H} -> VTGT
- R10 pad 2: Net-(U8-A) -> Net-(U4-A1)
- R11 pad 1: Net-(U8-B) -> Net-(U4-B1)
- R16 pad 1: /JTAG/VOUT -> /JTAG/T_TXD_EN
- R19 pad 1: VTGT -> Net-(U7-B)
- R19 pad 2: /JTAG/~{T_RESET_H} -> /JTAG/T_TCK_SWCLK_H
- R20 pad 2: Net-(U9-A) -> Net-(U8-A1)
- R21 pad 1: Net-(U9-B) -> Net-(U8-B1)
- R23 pad 2: Net-(U2-B) (its old number) -> /JTAG/T_TCK_SWCLK_H
- R24 pad 1: +3V3 -> /JTAG/T_TDO_SWO
- R24 pad 2: /MCU/~{DF_CS} -> Net-(U4-A2)
- R25 pad 1: Net-(U4-B) -> Net-(U4-B2)
- R31 pad 1: Net-(Q4-G) -> Net-(Q1-G)
- R46 pad 2: Net-(R33-Pad2) -> Net-(R46-Pad2)
- R47 pad 1: Net-(R33-Pad2) -> Net-(R46-Pad2)
- R47 pad 2: Net-(C14-Pad1) -> /RP2040N/KEY
- R6 pad 2: Net-(U6-A) (its old number) -> Net-(U8-A2)
- R7 pad 1: Net-(U6-B) (its old number) -> Net-(U8-B2)
- SW1 pad 1: Net-(R25-Pad1) -> Net-(D3-Pad3)
- SW1 pad 2: Net-(R26-Pad2) -> unconnected-(SW1-Pad2)
- SW1 pad 4: Net-(R27-Pad2) -> Net-(D2-Pad3)
- SW3 pad 1: Net-(R39-Pad2) -> Net-(R46-Pad2)
- U10 pad 3: Net-(U17-EN) -> unconnected-(U10-EN-Pad3)
- U13 pad 34: /JTAG/VOUT -> /JTAG/T_TXD_EN
- U15 pad 3: Net-(U11-EN) -> unconnected-(U15-EN-Pad3)
- U4 pad 2: GND -> Net-(U4-A1)
- U4 pad 3: Net-(U8-A) -> Net-(U4-A2)
- U4 pad 4: Net-(U8-B) -> GND
- U4 pad 6: VTGT -> Net-(U4-B2)
- U7 pad 4: Net-(U2-B) (its old number) -> Net-(U7-B)
- U8 pad 2: GND -> Net-(U8-A1)
- U8 pad 3: Net-(U9-A) -> Net-(U8-A2)
- U8 pad 4: Net-(U9-B) -> GND
- U8 pad 6: VTGT -> Net-(U8-B2)
Routing:
- net +3V3: track 122.2 -> 28.4 mm, vias 6 -> 5
- net +5V: track 73.0 -> 0.00 mm
- net Net-(U1-I2C1_SCL/ADC1/GP27): track 53.7 -> 0.00 mm
- net /JTAG/T_RXD: track 51.4 -> 0.00 mm
- net /JTAG/M_SWDIN: track 51.0 -> 0.00 mm, vias 1 -> 0
- net /JTAG/T_TMS_SWDIO: track 50.2 -> 0.00 mm, vias 1 -> 0
- net VTGT: track 50.5 -> 2.34 mm, vias 8 -> 5
- net /JTAG/T_TCK_SWCLK: track 47.8 -> 0.00 mm, vias 1 -> 0
- net /JTAG/~{T_RESET}: track 47.7 -> 0.00 mm
- net /JTAG/T_TXD: track 47.6 -> 0.00 mm
- net /JTAG/CTRL_5V: track 44.9 -> 0.00 mm, vias 1 -> 0
- net /JTAG/T_TDO_SWO: track 44.2 -> 0.00 mm, vias 1 -> 0
- net /JTAG/CTRL_3V3: track 36.4 -> 0.00 mm, vias 1 -> 0
- net /JTAG/T_TDI: track 31.7 -> 0.00 mm, vias 1 -> 0
- net GND: track 33.5 -> 5.38 mm, vias 7 -> 0
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Other:
- board size 82 x 30 mm -> 82 x 35 mm
