File: Hardware/rplink/rplink.kicad_sch (KiCad schematic)
At the start: 0 parts

Commit message: rev 0.1
Parts:
- added FID1: Fiducial, Fiducial:Fiducial_0.5mm_Mask1.5mm, symbol Mechanical:Fiducial
- added FID2, FID3: Fiducial, Fiducial:Fiducial_0.5mm_Mask1.5mm, symbol Generic:Fiducial
- added H1, H2, H3, H4: MountingHole, MountingHole:MountingHole_3.2mm_M3, symbol Mechanical:MountingHole
Other:
- removed sheet MCU
- added sheet PowerSupply (ps.kicad_sch)
- added sheet RP2040N (rp2404n.kicad_sch)
- sheet JTAG ports: added T_RESET_CHK, T_RESET_EN, T_RXD, T_SWDIN, T_SWD_OE, T_TCK_EN, T_TCK_SWCLK, T_TDI, T_TDI_EN, T_TDO_SWO, T_TMS_SWDIO, T_TXD, T_TXD_EN, ~{T_RESET}; removed none
